Commit message: added ros2_control gazebo

File: description/camera.xacro (robot description, xacro)
@@ -4,5 +4,5 @@
         <parent link="base_link" />
         <child link="camera_link" />
-        <origin xyz="0.305 0 0.08" rpy="0 0 0" />
+        <origin xyz="0.28 0 0" rpy="0 0 0" />
     </joint>
     <joint name="camera_optical_joint" type="fixed">

File: description/robot.urdf.xacro (robot description, xacro)
@@ -2,6 +2,7 @@
 <robot xmlns:xacro="http://www.ros.org/wiki/xacro" name="robot">
     <xacro:include filename="robot_core.xacro" />
-    <xacro:include filename="gazebo_control.xacro" />
+    <!-- <xacro:include filename="gazebo_control.xacro" /> -->
     <xacro:include filename="lidar.xacro" />
     <xacro:include filename="camera.xacro" />
+    <xacro:include filename="ros2_control.xacro" />
 </robot>

Commit message: camera orgin

File: description/camera.xacro (robot description, xacro)
@@ -4,5 +4,5 @@
         <parent link="base_link" />
         <child link="camera_link" />
-        <origin xyz="0.28 0 0" rpy="0 0 0" />
+        <origin xyz="0.2 0 0.075" rpy="0 0 0" />
     </joint>
     <joint name="camera_optical_joint" type="fixed">
