Commit message: Update lidar and robot core configurations: adjust lidar joint orientation and update update rate for sensor; add base footprint link and joint in robot_core.xacro; integrate SLAM node in launch file with appropriate parameters and remappings for enhanced simulation capabilities.

File: description/lidar.xacro (robot description, xacro)
@@ -1,60 +1,61 @@
 <?xml version="1.0"?>
 <robot xmlns:xacro="http://www.ros.org/wiki/xacro">
-    <link name="lidar_frame">
-        <visual>
-            <geometry>
-                <cylinder radius="0.05" length="0.04" />
-            </geometry>
-            <material name="red" />
-        </visual>
-        <collision>
-            <geometry>
-                <cylinder radius="0.05" length="0.04" />
-            </geometry>
-        </collision>
-        <xacro:inertial_cylinder mass="0.1" length="0.04" radius="0.05">
-            <origin xyz="0 0 0" rpy="0 0 0" />
-        </xacro:inertial_cylinder>
-    </link>
-    <joint name="lidar_joint" type="fixed">
-        <parent link="base_link" />
-        <child link="lidar_frame" />
-        <origin xyz="0.1 0 0.12" rpy="0 0 0" />
-    </joint>
-   <gazebo reference="lidar_frame">
+  <link name="lidar_frame">
+    <visual>
+      <geometry>
+        <cylinder radius="0.05" length="0.04" />
+      </geometry>
+      <material name="red" />
+    </visual>
+    <collision>
+      <geometry>
+        <cylinder radius="0.05" length="0.04" />
+      </geometry>
+    </collision>
+    <xacro:inertial_cylinder mass="0.1" length="0.04" radius="0.05">
+      <origin xyz="0 0 0" rpy="0 0 0" />
+    </xacro:inertial_cylinder>
+  </link>
+  <joint name="lidar_joint" type="fixed">
+    <parent link="base_link" />
+    <child link="lidar_frame" />
+    <origin xyz="0.2 0 0.12" rpy="0 0 3.14159" /> <!-- Rotated 180 degrees to face forward -->
+  </joint>
+  <gazebo reference="lidar_frame">
     <material>Gazebo/Red</material>
     <sensor name="laser" type="ray">
-        <pose>0 0 0 0 0 0</pose>
-        <visualize>true</visualize>
-        <update_rate>10</update_rate>
-        <ray>
-            <scan>
-                <horizontal>
-                    <samples>360</samples>
-                    <resolution>1</resolution>
-                    <min_angle>-3.14159265359</min_angle>
-                    <max_angle>3.14159265359</max_angle>
-                </horizontal>
-            </scan>
-            <range>
-                <min>0.15</min>
-                <max>12.0</max>
-                <resolution>0.03</resolution>
-            </range>
-        </ray>
-        <plugin name="laser_controller" filename="libgazebo_ros_ray_sensor.so">
-            <ros>
-                <namespace>/</namespace>
-                <remapping>~/out:=scan</remapping>
-                <qos>
-                    <reliability>best_effort</reliability>
-                    <history>keep_last</history>
-                    <depth>5</depth>
-                </qos>
-            </ros>
-            <output_type>sensor_msgs/LaserScan</output_type>
-            <frame_name>lidar_frame</frame_name>
-        </plugin>
+      <pose>0 0 0 0 0 0</pose>
+      <visualize>false</visualize>
+      <!-- Adjusted update rate to 5 Hz for RPLIDAR A1 typical operation -->
+      <update_rate>5</update_rate>
+      <ray>
+        <scan>
+          <horizontal>
+            <samples>360</samples>
+            <resolution>1</resolution>
+            <min_angle>-3.14159265359</min_angle>
+            <max_angle>3.14159265359</max_angle>
+          </horizontal>
+        </scan>
+        <range>
+          <min>0.15</min>
+          <max>12.0</max>
+          <resolution>0.03</resolution>
+        </range>
+      </ray>
+      <plugin name="laser_controller" filename="libgazebo_ros_ray_sensor.so">
+        <ros>
+          <namespace>/</namespace>
+          <remapping>~/out:=scan</remapping>
+          <qos>
+            <reliability>best_effort</reliability>
+            <history>keep_last</history>
+            <depth>5</depth>
+          </qos>
+        </ros>
+        <output_type>sensor_msgs/LaserScan</output_type>
+        <frame_name>lidar_frame</frame_name>
+      </plugin>
     </sensor>
-</gazebo>
+  </gazebo>
 </robot>

File: description/robot_core.xacro (robot description, xacro)
@@ -19,4 +19,12 @@
     <!-- BASE LINK -->
     <link name="base_link">
+    </link>
+    <!-- BASE FOOTPRINT LINK -->
+    <joint name="base_footprint_joint" type="fixed">
+        <parent link="base_link"/>
+        <child link="base_footprint"/>
+        <origin xyz="0 0 0"/>
+    </joint>
+    <link name="base_footprint">
     </link>
     <!-- CHASSIS LINK -->

Commit message: added - slam param fixed gazebo and lidar publish rate fixed odam ppublish - controller

File: description/lidar.xacro (robot description, xacro)
@@ -1,4 +1,5 @@
 <?xml version="1.0"?>
 <robot xmlns:xacro="http://www.ros.org/wiki/xacro">
+  <!-- LIDAR Visual and Physical Properties -->
   <link name="lidar_frame">
     <visual>
@@ -13,13 +14,16 @@
       </geometry>
     </collision>
+    <!-- Simple inertial properties for a fixed sensor -->
     <xacro:inertial_cylinder mass="0.1" length="0.04" radius="0.05">
       <origin xyz="0 0 0" rpy="0 0 0" />
     </xacro:inertial_cylinder>
   </link>
+  <!-- Mount LIDAR to the chassis -->
   <joint name="lidar_joint" type="fixed">
     <parent link="base_link" />
     <child link="lidar_frame" />
-    <origin xyz="0.2 0 0.12" rpy="0 0 3.14159" /> <!-- Rotated 180 degrees to face forward -->
+    <origin xyz="0.2 0 0.12" rpy="0 0 0" />
   </joint>
+  <!-- Improved RPLIDAR A1 Gazebo Configuration -->
   <gazebo reference="lidar_frame">
     <material>Gazebo/Red</material>
@@ -27,30 +31,28 @@
       <pose>0 0 0 0 0 0</pose>
       <visualize>false</visualize>
-      <!-- Adjusted update rate to 5 Hz for RPLIDAR A1 typical operation -->
-      <update_rate>5</update_rate>
+      <update_rate>10.0</update_rate>  <!-- Increased from 5.5 for more stable updates -->
       <ray>
         <scan>
           <horizontal>
-            <samples>360</samples>
+            <samples>720</samples>  <!-- Doubled from 360 for higher resolution -->
             <resolution>1</resolution>
-            <min_angle>-3.14159265359</min_angle>
-            <max_angle>3.14159265359</max_angle>
+            <min_angle>-3.14159</min_angle>
+            <max_angle>3.14159</max_angle>
           </horizontal>
         </scan>
         <range>
-          <min>0.15</min>
-          <max>12.0</max>
-          <resolution>0.03</resolution>
+          <min>0.15</min>  <!-- RPLIDAR A1 minimum range -->
+          <max>12.0</max>  <!-- RPLIDAR A1 maximum range -->
+          <resolution>0.01</resolution>  <!-- Improved from 0.03 -->
         </range>
+        <noise>
+          <type>gaussian</type>
+          <mean>0.0</mean>
+          <stddev>0.01</stddev>
+        </noise>
       </ray>
       <plugin name="laser_controller" filename="libgazebo_ros_ray_sensor.so">
         <ros>
-          <namespace>/</namespace>
           <remapping>~/out:=scan</remapping>
-          <qos>
-            <reliability>best_effort</reliability>
-            <history>keep_last</history>
-            <depth>5</depth>
-          </qos>
         </ros>
         <output_type>sensor_msgs/LaserScan</output_type>

File: description/robot_core.xacro (robot description, xacro)
@@ -18,10 +18,25 @@
     </material>
     <!-- BASE LINK -->
+    <!-- This is the actual physical base of the robot -->
     <link name="base_link">
+        <visual>
+            <geometry>
+                <box size="0.3 0.3 0.02"/>
+            </geometry>
+            <material name="white"/>
+        </visual>
+        <collision>
+            <geometry>
+                <box size="0.3 0.3 0.02"/>
+            </geometry>
+        </collision>
+        <xacro:inertial_box mass="0.5" x="0.3" y="0.3" z="0.02">
+            <origin xyz="0 0 0" rpy="0 0 0"/>
+        </xacro:inertial_box>
     </link>
     <!-- BASE FOOTPRINT LINK -->
     <joint name="base_footprint_joint" type="fixed">
-        <parent link="base_link"/>
-        <child link="base_footprint"/>
+        <parent link="base_footprint"/>
+        <child link="base_link"/>
         <origin xyz="0 0 0"/>
     </joint>

Commit message: Add LIDAR configuration in lidar.xacro file
This commit introduces a new XACRO file for the LIDAR sensor, defining its visual and physical properties, joint configuration, and Gazebo simulation settings. The LIDAR is mounted to the chassis with specified inertial properties and sensor parameters tailored for the RPLIDAR A1 model.

File: description/lidar.xacro (robot description, xacro)
@@ -23,5 +23,5 @@
     <parent link="base_link" />
     <child link="lidar_frame" />
-    <origin xyz="0.2 0 0.12" rpy="0 0 0" />
+    <origin xyz="0.0 0 0.08" rpy="0 0 0" />
   </joint>
   <!-- RPLIDAR A1 Gazebo Configuration -->
@@ -42,5 +42,5 @@
         </scan>
         <range>
-          <min>0.15</min>  <!-- RPLIDAR A1 minimum range -->
+          <min>0.2</min>  <!-- Adjusted to match real LiDAR -->
           <max>12.0</max>  <!-- RPLIDAR A1 maximum range -->
           <resolution>0.01</resolution>

Commit message: Add configuration files for EKF, controllers, LIDAR, and launch setup
- Created `ekf.yaml` for EKF filter parameters including sensor timeout and frame configurations.
- Added `my_controllers.yaml` for controller manager settings, including differential drive controller parameters.
- Introduced `lidar.xacro` for LIDAR model definition with visual and physical properties, including Gazebo integration.
- Implemented `launch_robot.launch.py` to set up the robot's launch configuration, including nodes for state publishing and controller management.

File: description/lidar.xacro (robot description, xacro)
@@ -23,5 +23,5 @@
     <parent link="base_link" />
     <child link="lidar_frame" />
-    <origin xyz="0.0 0 0.08" rpy="0 0 0" />
+    <origin xyz="0.15 0 0.12" rpy="0 0 0" />
   </joint>
   <!-- RPLIDAR A1 Gazebo Configuration -->

Commit message: Add LIDAR configuration files for TurtleBot3
- Introduced lidar.xacro to define the visual and physical properties of the LIDAR sensor, including its geometry, inertial properties, and Gazebo configuration.
- Created sllidar_a1_launch.launch.py to facilitate the launch of the LIDAR node with configurable parameters such as serial port and scan mode, along with static transforms for the robot's frame.

File: description/lidar.xacro (robot description, xacro)
@@ -2,30 +2,33 @@
 <robot xmlns:xacro="http://www.ros.org/wiki/xacro">
   <!-- LIDAR Visual and Physical Properties -->
-  <link name="lidar_frame">
+  <link name="laser_frame">
     <visual>
+      <origin xyz="0 0 0" rpy="0 0 0"/>
       <geometry>
-        <cylinder radius="0.05" length="0.04" />
+        <cylinder radius="0.035" length="0.010" />
       </geometry>
-      <material name="red" />
+      <material name="white" />
     </visual>
     <collision>
+      <origin xyz="0 0 0" rpy="0 0 0"/>
       <geometry>
-        <cylinder radius="0.05" length="0.04" />
+        <cylinder radius="0.035" length="0.010" />
       </geometry>
     </collision>
-    <!-- Simple inertial properties for a fixed sensor -->
-    <xacro:inertial_cylinder mass="0.1" length="0.04" radius="0.05">
-      <origin xyz="0 0 0" rpy="0 0 0" />
-    </xacro:inertial_cylinder>
+    <inertial>
+      <origin xyz="0 0 0" rpy="0 0 0"/>
+      <mass value="0.1"/>
+      <inertia ixx="0.000084" ixy="0.0" ixz="0.0" iyy="0.000084" iyz="0.0" izz="0.0000002"/>
+    </inertial>
   </link>
-  <!-- Mount LIDAR to the chassis -->
+  <!-- Mount LiDAR to the chassis -->
   <joint name="lidar_joint" type="fixed">
     <parent link="base_link" />
-    <child link="lidar_frame" />
-    <origin xyz="0.15 0 0.12" rpy="0 0 0" />
+    <child link="laser_frame" />
+    <origin xyz="0 0 0.105" rpy="0 0 0" />
   </joint>
-  <!-- RPLIDAR A1 Gazebo Configuration -->
-  <gazebo reference="lidar_frame">
-    <material>Gazebo/Red</material>
+  <!-- TurtleBot3 LiDAR Gazebo Configuration -->
+  <gazebo reference="laser_frame">
+    <material>Gazebo/White</material>
     <sensor name="laser" type="ray">
       <pose>0 0 0 0 0 0</pose>
@@ -35,5 +38,5 @@
         <scan>
           <horizontal>
-            <samples>360</samples>  <!-- Standard RPLIDAR A1 resolution -->
+            <samples>360</samples>
             <resolution>1</resolution>
             <min_angle>-3.14159</min_angle>
@@ -42,6 +45,6 @@
         </scan>
         <range>
-          <min>0.2</min>  <!-- Adjusted to match real LiDAR -->
-          <max>12.0</max>  <!-- RPLIDAR A1 maximum range -->
+          <min>0.1</min>
+          <max>30.0</max>
           <resolution>0.01</resolution>
         </range>
@@ -49,13 +52,10 @@
           <type>gaussian</type>
           <mean>0.0</mean>
-          <stddev>0.01</stddev>
+          <stddev>0.0</stddev>
         </noise>
       </ray>
-      <plugin name="laser_controller" filename="libgazebo_ros_ray_sensor.so">
-        <ros>
-          <remapping>~/out:=scan</remapping>
-        </ros>
-        <output_type>sensor_msgs/LaserScan</output_type>
-        <frame_name>lidar_frame</frame_name>
+      <plugin name="gazebo_ros_laser" filename="libgazebo_ros_laser.so">
+        <topicName>/scan</topicName>
+        <frameName>laser_frame</frameName>
       </plugin>
     </sensor>

Commit message: Add configuration files for robot controllers, lidar description, and launch scripts
- Created `my_controllers.yaml` to define parameters for joint state broadcaster and differential drive controller.
- Added `lidar.xacro` for lidar model including visual, collision, and inertial properties.
- Implemented `launch_robot.launch.py` to manage robot state publisher and controller nodes with improved timing.
- Introduced `sllidar_a1_launch.launch.py` for configuring and launching the SLLIDAR node with customizable parameters.

File: description/lidar.xacro (robot description, xacro)
@@ -1,5 +1,4 @@
 <?xml version="1.0"?>
 <robot xmlns:xacro="http://www.ros.org/wiki/xacro">
-  <!-- LIDAR Visual and Physical Properties -->
   <link name="laser_frame">
     <visual>
@@ -8,5 +7,5 @@
         <cylinder radius="0.035" length="0.010" />
       </geometry>
-      <material name="white" />
+      <material name="red" />
     </visual>
     <collision>
@@ -22,13 +21,11 @@
     </inertial>
   </link>
-  <!-- Mount LiDAR to the chassis -->
   <joint name="lidar_joint" type="fixed">
     <parent link="base_link" />
     <child link="laser_frame" />
-    <origin xyz="0 0 0.105" rpy="0 0 0" />
+    <origin xyz="0.20 0 0.100" rpy="0 0 0" />
   </joint>
-  <!-- TurtleBot3 LiDAR Gazebo Configuration -->
   <gazebo reference="laser_frame">
-    <material>Gazebo/White</material>
+    <material>Gazebo/Black</material>
     <sensor name="laser" type="ray">
       <pose>0 0 0 0 0 0</pose>
