Commit message: updated lauch file

File: description/robot_core.xacro (robot description, xacro)
@@ -1,16 +1,16 @@
 <?xml version="1.0"?>
-<robot xmlns:xacro="http://www.ros.org/wiki/xacro">
-    <xacro:include filename="inertial_macros.xacro" />
+<robot xmlns:xacro="http://www.ros.org/wiki/xacro" >
+    <xacro:include filename="inertial_macros.xacro"/>
     <material name="white">
         <color rgba="1 1 1 1" />
     </material>
     <material name="orange">
-        <color rgba="1 0.3 0.1 1" />
+        <color rgba="1 0.3 0.1 1"/>
     </material>
     <material name="blue">
-        <color rgba="0.2 0.2 1 1" />
+        <color rgba="0.2 0.2 1 1"/>
     </material>
     <material name="black">
-        <color rgba="0 0 0 1" />
+        <color rgba="0 0 0 1"/>
     </material>
     <!-- BASE LINK -->
@@ -19,24 +19,24 @@
     <!-- CHASSIS LINK -->
     <joint name="chassis_joint" type="fixed">
-        <parent link="base_link" />
-        <child link="chassis" />
-        <origin xyz="-0.1 0 0" rpy="0 0 0" />
+        <parent link="base_link"/>
+        <child link="chassis"/>
+        <origin xyz="-0.1 0 0"/>
     </joint>
     <link name="chassis">
         <visual>
-            <origin xyz="0.15 0 0.075" />
+            <origin xyz="0.15 0 0.075"/>
             <geometry>
-                <box size="0.3 0.3 0.15" />
+                <box size="0.3 0.3 0.15"/>
             </geometry>
-            <material name="white" />
+            <material name="white"/>
         </visual>
         <collision>
-            <origin xyz="0.15 0 0.075" />
+            <origin xyz="0.15 0 0.075"/>
             <geometry>
-                <box size="0.3 0.3 0.15" />
+                <box size="0.3 0.3 0.15"/>
             </geometry>
         </collision>
         <xacro:inertial_box mass="0.5" x="0.3" y="0.3" z="0.15">
-            <origin xyz="0.15 0 0.075" />
+            <origin xyz="0.15 0 0.075" rpy="0 0 0"/>
         </xacro:inertial_box>
     </link>
@@ -46,23 +46,23 @@
     <!-- LEFT WHEEL LINK -->
     <joint name="left_wheel_joint" type="continuous">
-        <parent link="base_link" />
-        <child link="left_wheel" />
+        <parent link="base_link"/>
+        <child link="left_wheel"/>
         <origin xyz="0 0.175 0" rpy="-${pi/2} 0 0" />
-        <axis xyz="0 0 1" />
+        <axis xyz="0 0 1"/>
     </joint>
     <link name="left_wheel">
         <visual>
             <geometry>
-                <cylinder radius="0.05" length="0.04" />
+                <cylinder radius="0.05" length="0.04"/>
             </geometry>
-            <material name="blue" />
+            <material name="blue"/>
         </visual>
         <collision>
             <geometry>
-                <cylinder radius="0.05" length="0.04" />
+                <cylinder radius="0.05" length="0.04"/>
             </geometry>
         </collision>
         <xacro:inertial_cylinder mass="0.1" length="0.04" radius="0.05">
-            <origin xyz="0 0 0" rpy="0 0 0" />
+            <origin xyz="0 0 0" rpy="0 0 0"/>
         </xacro:inertial_cylinder>
     </link>
@@ -72,23 +72,23 @@
     <!-- RIGHT WHEEL LINK -->
     <joint name="right_wheel_joint" type="continuous">
-        <parent link="base_link" />
-        <child link="right_wheel" />
+        <parent link="base_link"/>
+        <child link="right_wheel"/>
         <origin xyz="0 -0.175 0" rpy="${pi/2} 0 0" />
-        <axis xyz="0 0 -1" />
+        <axis xyz="0 0 -1"/>
     </joint>
     <link name="right_wheel">
         <visual>
             <geometry>
-                <cylinder radius="0.05" length="0.04" />
+                <cylinder radius="0.05" length="0.04"/>
             </geometry>
-            <material name="blue" />
+            <material name="blue"/>
         </visual>
         <collision>
             <geometry>
-                <cylinder radius="0.05" length="0.04" />
+                <cylinder radius="0.05" length="0.04"/>
             </geometry>
         </collision>
         <xacro:inertial_cylinder mass="0.1" length="0.04" radius="0.05">
-            <origin xyz="0 0 0" rpy="0 0 0" />
+            <origin xyz="0 0 0" rpy="0 0 0"/>
         </xacro:inertial_cylinder>
     </link>
@@ -98,28 +98,28 @@
     <!-- CASTER WHEEL LINK -->
     <joint name="caster_wheel_joint" type="fixed">
-        <parent link="chassis" />
-        <child link="caster_wheel" />
-        <origin xyz="0.24 0 0" />
+        <parent link="chassis"/>
+        <child link="caster_wheel"/>
+        <origin xyz="0.24 0 0"/>
     </joint>
     <link name="caster_wheel">
         <visual>
             <geometry>
-                <sphere radius="0.05" />
+                <sphere radius="0.05"/>
             </geometry>
-            <material name="black" />
+            <material name="black"/>
         </visual>
         <collision>
             <geometry>
-                <sphere radius="0.05" />
+                <sphere radius="0.05"/>
             </geometry>
         </collision>
         <xacro:inertial_sphere mass="0.1" radius="0.05">
-            <origin xyz="0 0 0" rpy="0 0 0" />
+            <origin xyz="0 0 0" rpy="0 0 0"/>
         </xacro:inertial_sphere>
     </link>
     <gazebo reference="caster_wheel">
         <material>Gazebo/Black</material>
-         <mu1 value="0.001" />
-        <mu2 value="0.001" />
+        <mu1 value="0.001"/>
+        <mu2 value="0.001"/>
     </gazebo>
 </robot>

Commit message: Add robot_core and ros2_control XACRO files for robot description and control

File: description/robot_core.xacro (robot description, xacro)
@@ -2,4 +2,8 @@
 <robot xmlns:xacro="http://www.ros.org/wiki/xacro" >
     <xacro:include filename="inertial_macros.xacro"/>
+    <!-- Wheel parameters -->
+    <xacro:property name="wheel_diameter" value="0.115"/> <!-- 11.5 cm -->
+    <xacro:property name="wheel_separation" value="0.255"/> <!-- 25.5 cm -->
+    <xacro:property name="wheel_radius" value="${wheel_diameter/2}"/>
     <material name="white">
         <color rgba="1 1 1 1" />
@@ -74,5 +78,5 @@
         <parent link="base_link"/>
         <child link="left_wheel"/>
-        <origin xyz="0 0.155 0" rpy="-${pi/2} 0 0" />
+        <origin xyz="0 ${wheel_separation/2} 0" rpy="-${pi/2} 0 0" />
         <axis xyz="0 0 1"/>
     </joint>
@@ -80,5 +84,5 @@
         <visual>
             <geometry>
-                <cylinder radius="0.055" length="0.04"/>
+                <cylinder radius="${wheel_radius}" length="0.04"/>
             </geometry>
             <material name="blue"/>
@@ -86,8 +90,8 @@
         <collision>
             <geometry>
-                <cylinder radius="0.055" length="0.04"/>
+                <cylinder radius="${wheel_radius}" length="0.04"/>
             </geometry>
         </collision>
-        <xacro:inertial_cylinder mass="0.1" length="0.04" radius="0.055">
+        <xacro:inertial_cylinder mass="0.1" length="0.04" radius="${wheel_radius}">
             <origin xyz="0 0 0" rpy="0 0 0"/>
         </xacro:inertial_cylinder>
@@ -100,5 +104,5 @@
         <parent link="base_link"/>
         <child link="right_wheel"/>
-        <origin xyz="0 -0.155 0" rpy="${pi/2} 0 0" />
+        <origin xyz="0 -${wheel_separation/2} 0" rpy="${pi/2} 0 0" />
         <axis xyz="0 0 -1"/>
     </joint>
@@ -106,5 +110,5 @@
         <visual>
             <geometry>
-                <cylinder radius="0.055" length="0.04"/>
+                <cylinder radius="${wheel_radius}" length="0.04"/>
             </geometry>
             <material name="blue"/>
@@ -112,8 +116,8 @@
         <collision>
             <geometry>
-                <cylinder radius="0.055" length="0.04"/>
+                <cylinder radius="${wheel_radius}" length="0.04"/>
             </geometry>
         </collision>
-        <xacro:inertial_cylinder mass="0.1" length="0.04" radius="0.055">
+        <xacro:inertial_cylinder mass="0.1" length="0.04" radius="${wheel_radius}">
             <origin xyz="0 0 0" rpy="0 0 0"/>
         </xacro:inertial_cylinder>

File: description/ros2_control.xacro (robot description, xacro)
@@ -31,5 +31,7 @@
           <param name="baud_rate">57600</param>
           <param name="timeout_ms">1000</param>
-          <param name="enc_counts_per_rev">1440</param>
+          <param name="encoder_ppr">7</param>
+          <param name="gear_ratio">99.5</param>
+          <param name="enc_counts_per_rev">697</param>
         </hardware>
       </xacro:unless>

Commit message: Add configuration files for robot parameters, description, and joystick launch

File: description/robot_core.xacro (robot description, xacro)
@@ -21,5 +21,13 @@
         <color rgba="1 0 0 1"/>
     </material>
+    <!-- BASE FOOTPRINT LINK -->
+    <link name="base_footprint">
+    </link>
     <!-- BASE LINK -->
+    <joint name="base_footprint_joint" type="fixed">
+        <parent link="base_footprint"/>
+        <child link="base_link"/>
+        <origin xyz="0 0 ${wheel_radius}"/>  <!-- Lift the robot by wheel radius -->
+    </joint>
     <!-- This is the actual physical base of the robot -->
     <link name="base_link">
@@ -38,12 +46,4 @@
             <origin xyz="0 0 0" rpy="0 0 0"/>
         </xacro:inertial_box>
-    </link>
-    <!-- BASE FOOTPRINT LINK -->
-    <joint name="base_footprint_joint" type="fixed">
-        <parent link="base_link"/>
-        <child link="base_footprint"/>
-        <origin xyz="0 0 0"/>
-    </joint>
-    <link name="base_footprint">
     </link>
     <!-- CHASSIS LINK -->

Commit message: Add configuration files for robot parameters, description, and launch setup
- Created `mapper_params_online_async.yaml` for SLAM toolbox parameters, enhancing outlier handling and optimization speed.
- Added `robot_core.xacro` to define the robot's structure, including chassis and wheel specifications.
- Introduced `launch_robot.launch.py` to manage robot launch configurations, including mock hardware options and improved timing for node initialization.

File: description/robot_core.xacro (robot description, xacro)
@@ -21,31 +21,6 @@
         <color rgba="1 0 0 1"/>
     </material>
-    <!-- BASE FOOTPRINT LINK -->
-    <link name="base_footprint">
-    </link>
-    <!-- BASE LINK -->
-    <joint name="base_footprint_joint" type="fixed">
-        <parent link="base_footprint"/>
-        <child link="base_link"/>
-        <origin xyz="0 0 ${wheel_radius}"/>  <!-- Lift the robot by wheel radius -->
-    </joint>
-    <!-- This is the actual physical base of the robot -->
-    <link name="base_link">
-        <visual>
-            <geometry>
-                <box size="0.3 0.3 0.02"/>
-            </geometry>
-            <material name="white"/>
-        </visual>
-        <collision>
-            <geometry>
-                <box size="0.3 0.3 0.02"/>
-            </geometry>
-        </collision>
-        <xacro:inertial_box mass="0.5" x="0.3" y="0.3" z="0.02">
-            <origin xyz="0 0 0" rpy="0 0 0"/>
-        </xacro:inertial_box>
-    </link>
     <!-- CHASSIS LINK -->
+    <link name="base_link"/>
     <joint name="chassis_joint" type="fixed">
         <parent link="base_link"/>

Commit message: Add configuration files and launch script for differential drive robot
- Created `my_controllers.yaml` to define controller parameters for the robot's joint state broadcaster and differential drive controller.
- Added `robot_core.xacro` to describe the robot's physical structure, including links and joints for the base, wheels, and caster wheel.
- Introduced `ros2_control.xacro` to configure the hardware interface for the robot, including parameters for mock and real hardware.
- Implemented `launch_robot.launch.py` to set up the launch process, including robot state publisher and controller manager with appropriate delays for initialization.

File: description/robot_core.xacro (robot description, xacro)
@@ -3,6 +3,6 @@
     <xacro:include filename="inertial_macros.xacro"/>
     <!-- Wheel parameters -->
-    <xacro:property name="wheel_diameter" value="0.11"/> <!-- 11.5 cm -->
-    <xacro:property name="wheel_separation" value="0.345"/> <!-- 34.5 cm -->
+    <xacro:property name="wheel_diameter" value="0.11"/> <!-- 11.0 cm -->
+    <xacro:property name="wheel_separation" value="0.32"/> <!-- 32.0 cm -->
     <xacro:property name="wheel_radius" value="${wheel_diameter/2}"/>
     <material name="white">

File: description/ros2_control.xacro (robot description, xacro)
@@ -21,5 +21,5 @@
                 <param name="baud_rate">115200</param>
                 <param name="timeout_ms">1000</param>
-                <param name="enc_counts_per_rev">2786</param>
+                <param name="enc_counts_per_rev">1393</param>
                 <param name="example_param_hw_start_duration_sec">0.0</param>
                 <param name="example_param_hw_stop_duration_sec">3.0</param>
