Commit message: Add DiffBot hardware interface and configuration files
- Created `diffbot_system.hpp` and `diffbot_system.cpp` to implement the hardware interface for the DiffBot, including methods for initialization, configuration, reading, and writing commands.
- Added `my_controllers.yaml` for configuring the controllers used by the DiffBot, specifying parameters such as wheel names, velocity limits, and update rates.
- Introduced `ros2_control.xacro` to define the robot's hardware configuration, including conditional loading for mock hardware and integration with Gazebo.

File: description/ros2_control.xacro (robot description, xacro)
@@ -1,64 +1,45 @@
 <?xml version="1.0"?>
 <robot xmlns:xacro="http://www.ros.org/wiki/xacro">
-  <xacro:arg name="use_mock_hardware" default="false"/>
-  <xacro:arg name="sim_mode" default="false"/>
-  <xacro:arg name="use_arduino" default="true"/>
-  <ros2_control name="DiffBotHardware" type="system">
-    <!-- Simulated Gazebo Plugin -->
-    <xacro:if value="$(arg sim_mode)">
-      <hardware>
-        <plugin>gazebo_ros2_control/GazeboSystem</plugin>
-      </hardware>
-    </xacro:if>
-    <!-- Mock Hardware Plugin -->
-    <xacro:if value="$(arg use_mock_hardware)">
-      <hardware>
-        <plugin>mock_components/GenericSystem</plugin>
-        <param name="calculate_dynamics">true</param>
-        <param name="left_wheel_name">left_wheel_joint</param>
-        <param name="right_wheel_name">right_wheel_joint</param>
-      </hardware>
-    </xacro:if>
-    <!-- Real Hardware Plugin -->
-    <xacro:unless value="$(arg sim_mode)">
-      <xacro:unless value="$(arg use_mock_hardware)">
-        <hardware>
-          <plugin>my_bot/DiffBotSystemHardware</plugin>
-          <param name="left_wheel_name">left_wheel_joint</param>
-          <param name="right_wheel_name">right_wheel_joint</param>
-          <param name="loop_rate">100.0</param>
-          <param name="device">/dev/ttyUSB0</param>
-          <param name="baud_rate">115200</param>
-          <param name="timeout_ms">1000</param>
-          <param name="enc_counts_per_rev">2787</param>
-        </hardware>
-      </xacro:unless>
-    </xacro:unless>
-    <!-- Joints -->
-    <joint name="left_wheel_joint">
-      <command_interface name="velocity">
-        <param name="min">-2.0</param>
-        <param name="max">2.0</param>
-      </command_interface>
-      <state_interface name="position"/>
-      <state_interface name="velocity"/>
-    </joint>
-    <joint name="right_wheel_joint">
-      <command_interface name="velocity">
-        <param name="min">-2.0</param>
-        <param name="max">2.0</param>
-      </command_interface>
-      <state_interface name="position"/>
-      <state_interface name="velocity"/>
-    </joint>
-  </ros2_control>
-  <!-- Gazebo plugin -->
-  <gazebo>
-    <plugin name="gazebo_ros2_control" filename="libgazebo_ros2_control.so">
-      <parameters>$(find my_bot)/config/my_controllers.yaml</parameters>
-      <robot_param>robot_description</robot_param>
-      <robot_param_node>robot_state_publisher</robot_param_node>
-      <update_rate>100.0</update_rate>
-    </plugin>
-  </gazebo>
+    <xacro:arg name="use_mock_hardware" default="false"/>
+    <xacro:arg name="sim_mode" default="false"/>
+    <xacro:property name="motor_power_multiplier" value="5.0"/>
+    <ros2_control name="RealRobot" type="system">
+        <xacro:if value="$(arg use_mock_hardware)">
+            <hardware>
+                <plugin>mock_components/GenericSystem</plugin>
+            </hardware>
+        </xacro:if>
+        <xacro:unless value="$(arg use_mock_hardware)">
+            <hardware>
+                <plugin>my_bot/DiffBotSystemHardware</plugin>
+                <param name="left_wheel_name">left_wheel_joint</param>
+                <param name="right_wheel_name">right_wheel_joint</param>
+                <param name="loop_rate">500.0</param>
+                <param name="device">/dev/ttyUSB0</param>
+                <param name="baud_rate">115200</param>
+                <param name="timeout_ms">1000</param>
+                <param name="enc_counts_per_rev">2000</param>
+                <param name="example_param_hw_start_duration_sec">0.0</param>
+                <param name="example_param_hw_stop_duration_sec">3.0</param>
+                <param name="motor_power_multiplier">${motor_power_multiplier}</param>
+            </hardware>
+        </xacro:unless>
+        <joint name="left_wheel_joint">
+            <command_interface name="velocity"/>
+            <state_interface name="position"/>
+            <state_interface name="velocity"/>
+        </joint>
+        <joint name="right_wheel_joint">
+            <command_interface name="velocity"/>
+            <state_interface name="position"/>
+            <state_interface name="velocity"/>
+        </joint>
+    </ros2_control>
+    <gazebo>
+        <plugin name="gazebo_ros2_control" filename="libgazebo_ros2_control.so">
+            <parameters>$(find my_bot)/config/my_controllers.yaml</parameters>
+            <robot_param>robot_description</robot_param>
+            <robot_param_node>robot_state_publisher</robot_param_node>
+        </plugin>
+    </gazebo>
 </robot>

Commit message: Add configuration files for robot control and parameters
- Created `my_controllers.yaml` to define controllers and parameters for the robot's joint state and differential drive.
- Added `ros2_control.xacro` to set up the robot's hardware interface, including joint definitions and Gazebo integration for simulation.

File: description/ros2_control.xacro (robot description, xacro)
@@ -4,4 +4,6 @@
     <xacro:arg name="sim_mode" default="false"/>
     <xacro:property name="motor_power_multiplier" value="5.0"/>
+    <xacro:property name="left_wheel_multiplier" value="-1.0"/>
+    <xacro:property name="right_wheel_multiplier" value="1.0"/>
     <ros2_control name="RealRobot" type="system">
         <xacro:if value="$(arg use_mock_hardware)">
@@ -23,4 +25,6 @@
                 <param name="example_param_hw_stop_duration_sec">3.0</param>
                 <param name="motor_power_multiplier">${motor_power_multiplier}</param>
+                <param name="left_wheel_multiplier">${left_wheel_multiplier}</param>
+                <param name="right_wheel_multiplier">${right_wheel_multiplier}</param>
             </hardware>
         </xacro:unless>

Commit message: Add configuration and description files for robot control and structure
- Created `my_controllers.yaml` to define parameters for joint state broadcasting and differential drive control.
- Added `robot_core.xacro` to describe the robot's physical structure, including links and joints for the base and wheels.
- Introduced `ros2_control.xacro` to set up the control system, including hardware configuration and joint interfaces for the robot's wheels.

File: description/ros2_control.xacro (robot description, xacro)
@@ -4,6 +4,4 @@
     <xacro:arg name="sim_mode" default="false"/>
     <xacro:property name="motor_power_multiplier" value="5.0"/>
-    <xacro:property name="left_wheel_multiplier" value="-1.0"/>
-    <xacro:property name="right_wheel_multiplier" value="1.0"/>
     <ros2_control name="RealRobot" type="system">
         <xacro:if value="$(arg use_mock_hardware)">
@@ -25,6 +23,4 @@
                 <param name="example_param_hw_stop_duration_sec">3.0</param>
                 <param name="motor_power_multiplier">${motor_power_multiplier}</param>
-                <param name="left_wheel_multiplier">${left_wheel_multiplier}</param>
-                <param name="right_wheel_multiplier">${right_wheel_multiplier}</param>
             </hardware>
         </xacro:unless>
