Commit message: Add configuration and launch files for robot simulation
- Introduced `mapper_params_online_async.yaml` for SLAM toolbox parameters.
- Added `gazebo_control.xacro` for Gazebo plugin configuration, including wheel and odometry settings.
- Created `robot_core.xacro` defining the robot's physical structure and materials.
- Implemented joystick control with `joystick.launch.py` for teleoperation.
- Developed `launch_sim.launch.py` to orchestrate the simulation environment, including static transforms and controller management.
- Added `rsp.launch.py` for robot state publishing and joint state management in simulation.

File: description/gazebo_control.xacro (robot description, xacro)
@@ -4,7 +4,7 @@
   <plugin name="diff_drive" filename="libgazebo_ros_diff_drive.so">
   <!-- Add these parameters -->
-  <update_rate>50</update_rate>
+  <update_rate>100</update_rate>
   <command_topic>cmd_vel</command_topic>
-  <publish_rate>50</publish_rate>
+  <publish_rate>100</publish_rate>
   <!-- Wheel Information-->
   <left_joint>left_wheel_joint</left_joint>
@@ -18,12 +18,18 @@
 <!-- The frame in which odometry data will be published. Expected value is the name of the odometry frame. -->
 <odometry_frame>odom</odometry_frame>
-<robot_base_frame>base_link</robot_base_frame>
+<robot_base_frame>base_footprint</robot_base_frame>
 <publish_odom>true</publish_odom>
 <publish_odom_tf>true</publish_odom_tf>
-<publish_wheel_tf>true</publish_wheel_tf>
+<publish_wheel_tf>false</publish_wheel_tf>
     <!-- Add this -->
     <ros>
         <use_sim_time>true</use_sim_time>
+        <!-- Added parameters to handle TF timing properly -->
+        <remapping>/tf:=tf</remapping>
+        <remapping>/tf_static:=tf_static</remapping>
     </ros>
+    <!-- Add parameters to fix wheel timing issues -->
+    <tf_future_dated_reads>true</tf_future_dated_reads>
+    <tf_message_filter_tolerance>0.1</tf_message_filter_tolerance>
   </plugin>
   </gazebo>

File: description/robot_core.xacro (robot description, xacro)
@@ -37,6 +37,6 @@
     <!-- BASE FOOTPRINT LINK -->
     <joint name="base_footprint_joint" type="fixed">
-        <parent link="base_footprint"/>
-        <child link="base_link"/>
+        <parent link="base_link"/>
+        <child link="base_footprint"/>
         <origin xyz="0 0 0"/>
     </joint>

Commit message: Add initial setup and configuration files for my_bot package
- Created setup.py for package configuration and dependencies.
- Added SLAM toolbox parameters in mapper_params_online_async.yaml.
- Included navigation parameters in nav2_params.yaml for AMCL and controller server.
- Defined robot description in gazebo_control.xacro and lidar.xacro.
- Established robot core structure in robot_core.xacro.
- Implemented launch file for simulation in launch_sim.launch.py.
- Created worlds for simulation: lidar.world and new.world.
- Configured various sensor and model properties for Gazebo simulation.

File: description/gazebo_control.xacro (robot description, xacro)
@@ -10,5 +10,5 @@
   <left_joint>left_wheel_joint</left_joint>
   <right_joint>right_wheel_joint</right_joint>
-  <wheel_separation>0.35</wheel_separation>
+  <wheel_separation>0.3</wheel_separation>
   <wheel_diameter>0.1</wheel_diameter>
 <!-- LIMITS-->

File: description/lidar.xacro (robot description, xacro)
@@ -22,5 +22,5 @@
     </inertial>
   </link>
-  <!-- Mount LiDAR to the chassis -->
+  <!-- Mount LiDAR to the base_link -->
   <joint name="lidar_joint" type="fixed">
     <parent link="base_link" />
@@ -34,5 +34,5 @@
       <pose>0 0 0 0 0 0</pose>
       <visualize>false</visualize>
-      <update_rate>10.0</update_rate>
+      <update_rate>20.0</update_rate>
       <ray>
         <scan>
@@ -58,4 +58,12 @@
         <topicName>/scan</topicName>
         <frameName>laser_frame</frameName>
+        <ros>
+          <remapping>~/out:=scan</remapping>
+          <qos>
+            <reliability>best_effort</reliability>
+            <history>keep_last</history>
+            <depth>5</depth>
+          </qos>
+        </ros>
       </plugin>
     </sensor>

File: description/robot_core.xacro (robot description, xacro)
@@ -3,6 +3,6 @@
     <xacro:include filename="inertial_macros.xacro"/>
     <!-- Wheel parameters -->
-    <xacro:property name="wheel_diameter" value="0.115"/> <!-- 11.5 cm -->
-    <xacro:property name="wheel_separation" value="0.255"/> <!-- 25.5 cm -->
+    <xacro:property name="wheel_diameter" value="0.11"/> <!-- 11.5 cm -->
+    <xacro:property name="wheel_separation" value="0.345"/> <!-- 34.5 cm -->
     <xacro:property name="wheel_radius" value="${wheel_diameter/2}"/>
     <material name="white">

Commit message: Add initial configuration and launch files for robot simulation
- Created `my_controllers.yaml` for controller parameters including joint state broadcaster and diff drive controller settings.
- Added `gazebo_control.xacro` for Gazebo integration with parameters for the diff drive plugin.
- Introduced `lidar.xacro` for LIDAR configuration, including visual and physical properties.
- Developed `robot_core.xacro` defining the robot's structure, including wheels, chassis, and base links.
- Implemented `ros2_control.xacro` for hardware interface and controller management.
- Established `launch_sim.launch.py` to orchestrate the simulation environment, including robot spawning and controller management.

File: description/gazebo_control.xacro (robot description, xacro)
@@ -10,5 +10,5 @@
   <left_joint>left_wheel_joint</left_joint>
   <right_joint>right_wheel_joint</right_joint>
-  <wheel_separation>0.3</wheel_separation>
+  <wheel_separation>0.42</wheel_separation>
   <wheel_diameter>0.1</wheel_diameter>
 <!-- LIMITS-->

File: description/lidar.xacro (robot description, xacro)
@@ -6,12 +6,12 @@
       <origin xyz="0 0 0" rpy="0 0 0"/>
       <geometry>
-        <cylinder radius="0.035" length="0.010" />
+        <cylinder radius="0.035" length="0.040" />
       </geometry>
-      <material name="white" />
+      <material name="black" />
     </visual>
     <collision>
       <origin xyz="0 0 0" rpy="0 0 0"/>
       <geometry>
-        <cylinder radius="0.035" length="0.010" />
+        <cylinder radius="0.035" length="0.040" />
       </geometry>
     </collision>
@@ -22,17 +22,18 @@
     </inertial>
   </link>
-  <!-- Mount LiDAR to the base_link -->
+  <!-- Mount LiDAR higher to avoid collision with chassis -->
   <joint name="lidar_joint" type="fixed">
     <parent link="base_link" />
     <child link="laser_frame" />
-    <origin xyz="0 0 0.105" rpy="0 0 0" />
+    <!-- Raised from 0.105 to 0.15 to clear the chassis -->
+    <origin xyz="0.1 0 0.15" rpy="0 0 0" />
   </joint>
-  <!-- TurtleBot3 LiDAR Gazebo Configuration -->
+  <!-- RPLIDAR A1 Gazebo Configuration -->
   <gazebo reference="laser_frame">
-    <material>Gazebo/White</material>
+    <material>Gazebo/Black</material>
     <sensor name="laser" type="ray">
       <pose>0 0 0 0 0 0</pose>
-      <visualize>false</visualize>
-      <update_rate>20.0</update_rate>
+      <visualize>true</visualize>
+      <update_rate>5.5</update_rate>
       <ray>
         <scan>
@@ -45,6 +46,6 @@
         </scan>
         <range>
-          <min>0.1</min>
-          <max>30.0</max>
+          <min>0.15</min>
+          <max>12.0</max>
           <resolution>0.01</resolution>
         </range>
@@ -52,18 +53,14 @@
           <type>gaussian</type>
           <mean>0.0</mean>
-          <stddev>0.0</stddev>
+          <stddev>0.01</stddev>
         </noise>
       </ray>
-      <plugin name="gazebo_ros_laser" filename="libgazebo_ros_laser.so">
-        <topicName>/scan</topicName>
-        <frameName>laser_frame</frameName>
+      <plugin name="gazebo_ros_ray_sensor" filename="libgazebo_ros_ray_sensor.so">
         <ros>
+          <namespace>/</namespace>
           <remapping>~/out:=scan</remapping>
-          <qos>
-            <reliability>best_effort</reliability>
-            <history>keep_last</history>
-            <depth>5</depth>
-          </qos>
         </ros>
+        <output_type>sensor_msgs/LaserScan</output_type>
+        <frame_name>laser_frame</frame_name>
       </plugin>
     </sensor>

File: description/robot_core.xacro (robot description, xacro)
@@ -32,18 +32,13 @@
     <!-- This is the actual physical base of the robot -->
     <link name="base_link">
+        <!-- Remove visual or make it a small reference point -->
         <visual>
             <geometry>
-                <box size="0.3 0.3 0.02"/>
+                <sphere radius="0.01"/>  <!-- Small sphere as reference -->
             </geometry>
-            <material name="white"/>
+            <material name="red"/>
         </visual>
-        <collision>
-            <geometry>
-                <box size="0.3 0.3 0.02"/>
-            </geometry>
-        </collision>
-        <xacro:inertial_box mass="0.5" x="0.3" y="0.3" z="0.02">
-            <origin xyz="0 0 0" rpy="0 0 0"/>
-        </xacro:inertial_box>
+        <!-- Remove any collision geometry from base_link -->
+        <!-- The chassis will handle all collisions -->
     </link>
     <!-- CHASSIS LINK -->

File: description/ros2_control.xacro (robot description, xacro)
@@ -3,37 +3,39 @@
     <xacro:arg name="use_mock_hardware" default="false"/>
     <xacro:arg name="sim_mode" default="false"/>
-    <xacro:property name="motor_power_multiplier" value="5.0"/>
-    <xacro:property name="left_wheel_multiplier" value="-1.0"/>
-    <xacro:property name="right_wheel_multiplier" value="1.0"/>
-    <ros2_control name="RealRobot" type="system">
-        <xacro:if value="$(arg use_mock_hardware)">
-            <hardware>
-                <plugin>mock_components/GenericSystem</plugin>
-            </hardware>
-        </xacro:if>
-        <xacro:unless value="$(arg use_mock_hardware)">
-            <hardware>
-                <plugin>my_bot/DiffBotSystemHardware</plugin>
-                <param name="left_wheel_name">left_wheel_joint</param>
-                <param name="right_wheel_name">right_wheel_joint</param>
-                <param name="loop_rate">100.0</param>
-                <param name="device">/dev/ttyUSB0</param>
-                <param name="baud_rate">115200</param>
-                <param name="timeout_ms">1000</param>
-                <param name="enc_counts_per_rev">1393</param>
-                <param name="example_param_hw_start_duration_sec">0.0</param>
-                <param name="example_param_hw_stop_duration_sec">3.0</param>
-                <param name="motor_power_multiplier">${motor_power_multiplier}</param>
-                <param name="left_wheel_multiplier">${left_wheel_multiplier}</param>
-                <param name="right_wheel_multiplier">${right_wheel_multiplier}</param>
-            </hardware>
-        </xacro:unless>
+    <ros2_control name="GazeboSystem" type="system">
+        <hardware>
+            <xacro:if value="$(arg sim_mode)">
+                <plugin>gazebo_ros2_control/GazeboSystem</plugin>
+            </xacro:if>
+            <xacro:unless value="$(arg sim_mode)">
+                <xacro:if value="$(arg use_mock_hardware)">
+                    <plugin>mock_components/GenericSystem</plugin>
+                </xacro:if>
+                <xacro:unless value="$(arg use_mock_hardware)">
+                    <plugin>my_bot/DiffBotSystemHardware</plugin>
+                    <param name="left_wheel_name">left_wheel_joint</param>
+                    <param name="right_wheel_name">right_wheel_joint</param>
+                    <param name="loop_rate">100.0</param>
+                    <param name="device">/dev/ttyUSB0</param>
+                    <param name="baud_rate">115200</param>
+                    <param name="timeout_ms">1000</param>
+                    <param name="enc_counts_per_rev">1393</param>
+                    <param name="motor_power_multiplier">5.0</param>
+                </xacro:unless>
+            </xacro:unless>
+        </hardware>
         <joint name="left_wheel_joint">
-            <command_interface name="velocity"/>
+            <command_interface name="velocity">
+                <param name="min">-10</param>
+                <param name="max">10</param>
+            </command_interface>
             <state_interface name="position"/>
             <state_interface name="velocity"/>
         </joint>
         <joint name="right_wheel_joint">
-            <command_interface name="velocity"/>
+            <command_interface name="velocity">
+                <param name="min">-10</param>
+                <param name="max">10</param>
+            </command_interface>
             <state_interface name="position"/>
             <state_interface name="velocity"/>
